File: PCB/example.kicad_pcb (KiCad board)
At the start: 2 copper layers, 47.6 x 63.8 mm, 7 parts, among them SW1 SW_Push, SW2 SW_Push, SW3 SW_Push, SW4 SW_Push, U1 XIAO-RP2040-DIP

Commit message: laptop
Parts:
- removed U1: XIAO-RP2040-DIP, OPL:XIAO-RP2040-DIP
- added SW5: SW_Push, Button_Switch_Keyboard:SW_Cherry_MX_1.00u_PCB, F.Cu at (145.4, 75.9)
- added SW6: SW_Push, Button_Switch_Keyboard:SW_Cherry_MX_1.00u_PCB, F.Cu at (107.3, 94.9)
- added SW7: SW_Push, Button_Switch_Keyboard:SW_Cherry_MX_1.00u_PCB, F.Cu at (126.4, 94.9)
- added SW8: SW_Push, Button_Switch_Keyboard:SW_Cherry_MX_1.00u_PCB, F.Cu at (145.4, 94.9)
- added SW9: RotaryEncoder, Rotary_Encoder:RotaryEncoder_Alps_EC11E-Switch_Vertical_H20mm_CircularMountingHoles, F.Cu at (136.0, 59.2)
- moved D2 79.2 mm to (113.7, 45.5)
- moved SW2 63.3 mm to (126.4, 56.8)
- moved SW4 63.3 mm to (126.4, 75.9)
- moved SW1 63.3 mm to (107.3, 56.8)
- moved SW3 63.3 mm to (107.3, 75.9)
- moved D1 48.6 mm to (113.7, 40.4)
Routing:
- net GND: track 104.7 -> 0.00 mm
- net Net-(D1-DOUT): track 53.7 -> 0.00 mm
- net Net-(D1-VDD): track 45.4 -> 0.00 mm
- net Net-(U1-GPIO4/MISO): track 44.7 -> 0.00 mm, vias 1 -> 0
- net Net-(U1-GPIO3/MOSI): track 42.7 -> 0.00 mm
- net Net-(U1-GPIO1/RX): track 27.5 -> 0.00 mm, vias 1 -> 0
- net Net-(U1-GPIO2/SCK): track 14.6 -> 0.00 mm
- net Net-(D1-DIN): track 7.99 -> 0.00 mm
- net +5V: track 1.08 -> 0.00 mm
Other:
- board outline removed
- board text removed: "Derp's Thingy"
- board text removed: "XIAO HERE"

Commit message: FIfrth commit
Parts:
- added U1: XIAO-RP2040-DIP, OPL Lib:XIAO-RP2040-DIP, F.Cu at (123.8, 39.6)
- moved D2 28.3 mm to (140.8, 37.4)
- moved D1 7.42 mm to (106.7, 37.7)
Routing:
- net GND: track 0.00 -> 197.5 mm, vias 0 -> 6
- net Net-(U1-GPIO26/ADC0/A0): track 0.00 -> 105.0 mm, vias 0 -> 3
- net Net-(U1-GPIO29/ADC3/A3): track 0.00 -> 95.2 mm, vias 0 -> 1
- net Net-(U1-GPIO27/ADC1/A1): track 0.00 -> 85.9 mm, vias 0 -> 1
- net Net-(U1-GPIO4/MISO): track 0.00 -> 67.3 mm, vias 0 -> 1
- net Net-(U1-GPIO28/ADC2/A2): track 0.00 -> 66.9 mm, vias 0 -> 3
- net Net-(D1-DOUT): track 0.00 -> 50.6 mm
- net Net-(U1-GPIO3/MOSI): track 0.00 -> 49.4 mm, vias 0 -> 1
- net Net-(D1-VDD): track 0.00 -> 42.5 mm
- net Net-(U1-GPIO1/RX): track 0.00 -> 35.5 mm
- net Net-(U1-GPIO0/TX): track 0.00 -> 30.5 mm, vias 0 -> 2
- net Net-(U1-GPIO2/SCK): track 0.00 -> 27.3 mm, vias 0 -> 1
- net Net-(U1-GPIO7/SCL): track 0.00 -> 25.8 mm, vias 0 -> 1
- net Net-(D1-DIN): track 0.00 -> 9.21 mm
Other:
- board outline added: 62.7 x 84.6 mm
- board text added: "Derp's Macro"
