File: PCB/example.kicad_sch (KiCad schematic)
At the start: 7 parts, among them SW1 SW_Push, SW2 SW_Push, SW3 SW_Push, SW4 SW_Push, U1 XIAO-RP2040-DIP

Commit message: laptop
Parts:
- added SW5, SW6, SW7, SW8: SW_Push, Button_Switch_Keyboard:SW_Cherry_MX_1.00u_PCB, symbol Switch:SW_Push
- added SW9: RotaryEncoder, Rotary_Encoder:RotaryEncoder_Alps_EC11E-Switch_Vertical_H20mm_CircularMountingHoles, symbol Device:RotaryEncoder
Connections:
- net GND: now also SW5.1, SW6.1, SW7.1, SW8.1, SW9.C
- net at U1.1 (GPIO26/ADC0/A0): now also SW5.2
- net at U1.2 (GPIO27/ADC1/A1): now also SW6.2
- net at U1.3 (GPIO28/ADC2/A2): now also SW7.2
- net at U1.4 (GPIO29/ADC3/A3): now also SW8.2
- net at U1.6 (GPIO7/SCL): now also SW9.A
- net at U1.7 (GPIO0/TX): now also SW9.B

Commit message: FIfrth commit
Parts:
- U1: footprint OPL:XIAO-RP2040-DIP -> OPL Lib:XIAO-RP2040-DIP
Changed lines of the file:
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@@
 			)
 		)
-		(property "Footprint" "OPL:XIAO-RP2040-DIP"
+		(property "Footprint" "OPL Lib:XIAO-RP2040-DIP"
 			(at 123.698 116.078 0)
 			(effects
